Commit message: Improve RViz launch and add production README

File: ack.urdf.xacro (robot description, xacro)
@@ -38,4 +38,13 @@
       <inertia ixx="0.0000003" ixy="0" ixz="0" iyy="0.0000006" iyz="0" izz="0.0000003" />
     </inertial>
+    <visual>
+      <origin xyz="0 0 0" rpy="0 0 0" />
+      <geometry>
+        <sphere radius="0.012"/>
+      </geometry>
+      <material name="silver">
+        <color rgba="0.7 0.7 0.7 1" />
+      </material>
+    </visual>
   </link>
   <joint name="FL_STEERING_JOINT" type="revolute">
@@ -79,4 +88,13 @@
       <inertia ixx="0.0000003" ixy="0" ixz="0" iyy="0.000001" iyz="0" izz="0.0000007" />
     </inertial>
+    <visual>
+      <origin xyz="0 0 0" rpy="0 0 0" />
+      <geometry>
+        <sphere radius="0.012"/>
+      </geometry>
+      <material name="silver">
+        <color rgba="0.7 0.7 0.7 1" />
+      </material>
+    </visual>
   </link>
   <joint name="FR_STEERING_JOINT" type="revolute">
@@ -253,5 +271,5 @@
   <gazebo>
     <plugin filename="ign_ros2_control::IgnRos2ControlPlugin" name="ign_ros2_control::IgnRos2ControlPlugin">
-      <ros_control_config_file>$(find ackermann_robot)/config/ackermann_control.yaml</ros_control_config_file>
+      <ros_control_config_file>/ackermann_ws/src/ackermann_robot/config/ackermann_control.yaml</ros_control_config_file>
     </plugin>
   </gazebo>
